Commit message: Update 2wd_properties.urdf.xacro

File: linorobot2_description/urdf/2wd_properties.urdf.xacro (robot description, xacro)
@@ -1,25 +1,19 @@
 <?xml version="1.0"?>
 <robot xmlns:xacro="http://ros.org/wiki/xacro">
-  <xacro:property name="base_length" value="0.24" />
-  <xacro:property name="base_width" value="0.275" />
-  <xacro:property name="base_height" value="0.003" />
+  <xacro:property name="base_length" value="0.4" />
+  <xacro:property name="base_width" value="0.44" />
+  <xacro:property name="base_height" value="0.10" />
   <xacro:property name="base_mass" value="1" />
-  <xacro:property name="wheel_radius" value="0.045" />
-  <xacro:property name="wheel_width" value="0.01" />
+  <xacro:property name="wheel_radius" value="0.05" />
+  <xacro:property name="wheel_width" value="0.02" />
   <xacro:property name="wheel_pos_x" value="0.0" />
-  <xacro:property name="wheel_pos_y" value="0.13" />
-  <xacro:property name="wheel_pos_z" value="-0.03" />
-  <xacro:property name="wheel_mass" value=".1" />
+  <xacro:property name="wheel_pos_y" value="0.195" />
+  <xacro:property name="wheel_pos_z" value="-0.09" />
+  <xacro:property name="wheel_mass" value="0.1" />
   <xacro:property name="wheel_torque" value="20" />
   <xacro:property name="front_caster_wheel" value="true" />
   <xacro:property name="rear_caster_wheel" value="true" />
   <xacro:property name="laser_pose">
-    <origin xyz="0.12 0 0.33" rpy="0 0 0"/>
-  </xacro:property>
-  <xacro:property name="depth_sensor_pose">
-    <origin xyz="0.14 0.0 0.045" rpy="0 0 0"/>
-  </xacro:property>
-  <xacro:property name="sonar_pose">
-    <origin xyz="0.15 0 0" rpy="0 0 0"/>
+    <origin xyz="0.18 0 0.11" rpy="0 0 0"/>
   </xacro:property>
 </robot>
